File: Hnah40-Atmega328p/PCB_V1/PCB/PCB.kicad_pcb (KiCad board)
At the start: 2 copper layers, 228.6 x 76.2 mm, 120 parts, among them J1 AVR-ISP-10, J2 Conn_01x05_Female, SW1 SW_PUSH, SW10 W, SW11 S, SW12 X, SW13 ALT, SW14 E, SW15 D, SW16 C, SW17 LEFT SPACE, SW18 R, SW19 F, SW2 ESC, SW20 V, SW21 T, SW22 G, SW23 B, SW24 RIGHT SPACE, SW25 Y, SW26 H, SW27 N, SW28 U, SW29 J, SW3 TAB, SW30 M, SW31 APP, SW32 I, SW33 K, SW34 ,, SW35 FN, SW36 O, SW37 L, SW38 BSPC, SW39 P, SW4 SHIFT, SW40 ENTER, SW41 SHIFT, SW42 CTRL, SW43 ., SW5 CTRL, SW6 Q, SW7 A, SW8 Z, SW9 WIN, U1 ATmega328-AU, U2 arduino-pro-mini, Y1 16MHz

Commit message: Watermark update
Parts:
- removed R1, R2: 4K7, Footprint_hnah87:R_0805_2012Metric
- added G***: LOGO, Footprint_hnah87:QR_code-m-me-HnahKB_solder_mask.8x8, B.Cu at (20.2, 41.9)
- added G***: LOGO, Footprint_hnah87:QR_code-m-me-HnahKB_solder_mask, F.Cu at (113.1, 56.6)
Routing:
- net GND: track 87.5 -> 89.9 mm, vias 110 -> 107
- net VCC: track 289.6 -> 287.6 mm
Other:
- board text added: "Hnah40 built by:"
