File: Hpad_4x5RGB/PCB/PCB.sch (KiCad schematic (older format))
At the start: 126 parts, among them J1 AVR-ISP-6, J10 Conn_4P_FM, J2 1x1_fm, J3 1x1_fm, J4 Conn_4P_FM, J5 Conn_4P_FM, J6 1x1_fm, J7 1x1_fm, J8 Conn_4P_FM, J9 01x05_fm, Q1 PZT2222A, SW1 Bootloader, SW10 SW_Push, SW11 SW_Push, SW12 SW_Push, SW13 SW_Push, SW14 SW_Push, SW15 SW_Push, SW16 SW_Push, SW17 SW_Push, SW18 SW_Push, SW19 SW_Push, SW2 SW_Push, SW20 SW_Push, SW21 SW_Push, SW22 SW_Push, SW23 SW_Push, SW24 SW_Push, SW25 SW_Push, SW26 SW_Push, SW27 SW_Push, SW28 SW_Push, SW3 SW_Push, SW4 SW_Push, SW5 SW_Push, SW6 SW_Push, SW7 SW_Push, SW8 SW_Push, SW9 SW_Push, U1 ATmega32U4-MU, U2 AP1117-50, U3 WS2811, Y1 16mhz

Commit message: missing wire fix
Parts:
- D12, D13, D14, D15, D16, D21, D22, D23, D24, D25, D3, D30, D31, D32, D33, D34, D4, D42, D43, D44, D45, D5, D6, D7: footprint Diode_SMD:D_SOD-323_HandSoldering -> Footprint_hnah87:D_SOD-323_HandSoldering
- USB1: symbol hro-type-c-31-m-12:HRO-TYPE-C-31-M-12-hro-type-c-31-m-12 -> PCB-rescue:HRO-TYPE-C-31-M-12-hro-type-c-31-m-12-hro-type-c-31-m-12
Connections:
- net GND: now also J10.4 (Pin_4)
- net Row6: now also U1.25 (PD4)
- removed net D4: J10.4 (Pin_4), U1.25 (PD4)
Other:
- moved on the sheet: BZ1, C4, D53, D54, D55, H1, H10, H2, H3, H4, H5, H6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
